File: KIcad/car_auto/car_auto.kicad_sch (KiCad schematic)
At the start: 10 parts, among them J1 PONTE-H, J2 HMC5883L, J3 NEO-6M, J4 ALIMENTAÇÃO, U1 ESP32-DEVKITC-32D, U2 ZC142200

Commit message: feat: Implementação da classe para controle dos motores via Bluetooth.
Parts:
- removed J3: NEO-6M, importados:JST_B4P-VH_LF__SN_, symbol importados:B4P-VH_LF__SN_
- removed U2: ZC142200, importados:MODULE_ZC142200, symbol importados:ZC142200
- added R1: 1.8k, Resistor_THT:R_Axial_DIN0207_L6.3mm_D2.5mm_P10.16mm_Horizontal, symbol Device:R
- added R2: 3.3k, Resistor_THT:R_Axial_DIN0207_L6.3mm_D2.5mm_P10.16mm_Horizontal, symbol Device:R
- added SW1: MTS-102, importados:MTS-102, symbol importados:MTS-102
- added U3: ~, importados:NEO-6M-V2-GPSMODULE-FOOTPRINT, symbol importados:NEO6MV2
Connections:
- net GND: now also R2.2, SW1.3, U3.4 (GND)
- net GPS-RX: now also U3.3 (TX)
- net GPS-TX: now also U3.2 (RX)
- net VCC: now also SW1.1, U3.1 (VCC)
- net enable: now reaches U1.J3-2 (IO23)
- net sinal_controle: now reaches U1.J3-8 (IO19)
- net sinal_controle: now also R1.1, R2.1
- new net: R1.2, SW1.2
Other:
- note added: "CHAVE MODO DE CONTROLE"
- note removed: "MÓDULO BLUETHOOT PARA CONTROLE REMOTO"
