File: KIcad/car_auto/localizacao_car/localizacao_car.kicad_pcb (KiCad board)
At the start: 2 copper layers, 96 x 96 mm, 6 parts, among them J1 B4P-VH_LF__SN_

Commit message: feat: Implementação da classe para controle dos motores via Bluetooth.
Parts:
- removed J1: B4P-VH_LF__SN_, importados:JST_B4P-VH_LF__SN_
- removed U1: ~, importados:NEO-6M-V2-GPSMODULE-FOOTPRINT
Routing:
- net Net-(U1-VCC): track 45.9 -> 0.00 mm
- net Net-(U1-RX): track 45.4 -> 0.00 mm
- net Net-(U1-TX): track 44.8 -> 0.00 mm
- net Net-(U1-GND): track 44.2 -> 0.00 mm
- net (no net): vias 4 -> 0
- added copper zone on B.Cu, net (none)
Other:
- outline, holes or cut-outs redrawn
