File: KIcad/car_auto/localizacao_car/localizacao_car.kicad_sch (KiCad schematic)
At the start: 6 parts, among them J1 B4P-VH_LF__SN_

Commit message: feat: Implementação da classe para controle dos motores via Bluetooth.
Parts:
- removed J1: B4P-VH_LF__SN_, importados:JST_B4P-VH_LF__SN_, symbol importados:B4P-VH_LF__SN_
- removed U1: ~, importados:NEO-6M-V2-GPSMODULE-FOOTPRINT, symbol importados:NEO6MV2
